Commit message: update xacro in order to use mobile base info yaml file

File: effibote3_description/urdf/effibote3.xacro (robot description, xacro)
@@ -4,45 +4,39 @@
     <xacro:include filename="$(find romea_mobile_base_description)/urdf/4WD_chassis.xacro" />
     <xacro:include filename="$(find romea_mobile_base_description)/ros2_control/4WD.ros2_control.xacro"/>
-    <xacro:property name="chassis_conf" value="$(find effibote3_description)/config/effibote3_chassis.yaml" />
-    <xacro:property name="kinematic_conf" value="$(find effibote3_description)/config/effibote3_kinematic.yaml" />
-    <xacro:property name="joints_conf_file" value="$(find effibote3_description)/config/effibote3_joints.yaml" />
-    <xacro:property name="links_conf_file" value="$(find effibote3_description)/config/effibote3_links.yaml" />
-    <xacro:property name="chassis_props" value="${load_yaml(chassis_conf)}"/>
-    <xacro:property name="kinematic_props" value="${load_yaml(kinematic_conf)}"/>
-    <xacro:property name="joints" value="${load_yaml(joints_conf_file)}"/>
-    <xacro:property name="links" value="${load_yaml(links_conf_file)}"/>
+    <xacro:property name="conf" value="$(find effibote3_description)/config/effibote3.yaml" />
+    <xacro:property name="props" value="${load_yaml(conf)['/**']['ros__parameters']['base_info']}" />
     <!-- Link names -->
-    <xacro:property name="base_link" value="${links['base_link_name']}" />
-    <xacro:property name="base_footprint_link" value="${links['base_footprint_link_name']}" />
-    <xacro:property name="inertial_link" value="${links['inertial_link_name']}" />
-    <xacro:property name="front_left_wheel_spinning_link" value="${links['front_left_wheel_spinning_link_name']}" />
-    <xacro:property name="front_right_wheel_spinning_link" value="${links['front_right_wheel_spinning_link_name']}" />
-    <xacro:property name="rear_left_wheel_spinning_link" value="${links['rear_left_wheel_spinning_link_name']}" />
-    <xacro:property name="rear_right_wheel_spinning_link" value="${links['rear_right_wheel_spinning_link_name']}" />
+    <xacro:property name="base_link" value="${props['links']['base_link_name']}" />
+    <xacro:property name="base_footprint_link" value="${props['links']['base_footprint_link_name']}" />
+    <xacro:property name="inertial_link" value="${props['links']['inertial_link_name']}" />
+    <xacro:property name="front_left_wheel_spinning_link" value="${props['links']['front_left_wheel_spinning_link_name']}" />
+    <xacro:property name="front_right_wheel_spinning_link" value="${props['links']['front_right_wheel_spinning_link_name']}" />
+    <xacro:property name="rear_left_wheel_spinning_link" value="${props['links']['rear_left_wheel_spinning_link_name']}" />
+    <xacro:property name="rear_right_wheel_spinning_link" value="${props['links']['rear_right_wheel_spinning_link_name']}" />
     <!-- Joint names -->
-    <xacro:property name="base_footprint_joint" value="${joints['base_footprint_joint_name']}" />
-    <xacro:property name="inertial_joint" value="${joints['inertial_joint_name']}" />
-    <xacro:property name="front_left_wheel_spinning_joint" value="${joints['front_left_wheel_spinning_joint_name']}" />
-    <xacro:property name="front_right_wheel_spinning_joint" value="${joints['front_right_wheel_spinning_joint_name']}" />
-    <xacro:property name="rear_left_wheel_spinning_joint" value="${joints['rear_left_wheel_spinning_joint_name']}" />
-    <xacro:property name="rear_right_wheel_spinning_joint" value="${joints['rear_right_wheel_spinning_joint_name']}" />
+    <xacro:property name="base_footprint_joint" value="${props['joints']['base_footprint_joint_name']}" />
+    <xacro:property name="inertial_joint" value="${props['joints']['inertial_joint_name']}" />
+    <xacro:property name="front_left_wheel_spinning_joint" value="${props['joints']['front_left_wheel_spinning_joint_name']}" />
+    <xacro:property name="front_right_wheel_spinning_joint" value="${props['joints']['front_right_wheel_spinning_joint_name']}" />
+    <xacro:property name="rear_left_wheel_spinning_joint" value="${props['joints']['rear_left_wheel_spinning_joint_name']}" />
+    <xacro:property name="rear_right_wheel_spinning_joint" value="${props['joints']['rear_right_wheel_spinning_joint_name']}" />
     <!-- Base Properties -->
-    <xacro:property name="aabb_length" value="${chassis_props['aabb']['length']}" />
-    <xacro:property name="aabb_width" value="${chassis_props['aabb']['width']}" />
-    <xacro:property name="aabb_height" value="${chassis_props['aabb']['height']}" />
-    <xacro:property name="wheelbase" value="${chassis_props['wheelbase']}"/>
-    <xacro:property name="front_track" value="${chassis_props['wheel_track']['front']}"/>
-    <xacro:property name="rear_track" value="${chassis_props['wheel_track']['rear']}"/>
-    <xacro:property name="mass_base" value="${chassis_props['mass']}" />
-    <xacro:property name="mass_center_x" value="${chassis_props['mass_center_position'][0]}" />
-    <xacro:property name="mass_center_y" value="${chassis_props['mass_center_position'][1]}" />
-    <xacro:property name="mass_center_z" value="${chassis_props['mass_center_position'][2]}" />
-    <xacro:property name="maximal_wheel_speed" value="${kinematic_props['maximal_wheel_speed']}"/>
-    <xacro:property name="body_reference_x" value="${kinematic_props['body_reference_x']}" />
+    <xacro:property name="aabb_length" value="${props['geometry']['aabb']['length']}" />
+    <xacro:property name="aabb_width" value="${props['geometry']['aabb']['width']}" />
+    <xacro:property name="aabb_height" value="${props['geometry']['aabb']['height']}" />
+    <xacro:property name="wheelbase" value="${props['geometry']['axles_distance']}"/>
+    <xacro:property name="front_track" value="${props['geometry']['front_axle']['wheels_distance']}"/>
+    <xacro:property name="rear_track" value="${props['geometry']['rear_axle']['wheels_distance']}"/>
+    <xacro:property name="mass_base" value="${props['inertia']['mass']}" />
+    <xacro:property name="mass_center_x" value="${props['inertia']['center'][0]}" />
+    <xacro:property name="mass_center_y" value="${props['inertia']['center'][1]}" />
+    <xacro:property name="mass_center_z" value="${props['inertia']['center'][2]}" />
+    <xacro:property name="maximal_wheel_speed" value="${props['wheels_speed_control']['command']['maximal_speed']}"/>
+    <xacro:property name="body_reference_x" value="${props['control_point'][0]}" />
     <!-- Wheel Properties -->
-    <xacro:property name="front_wheel_radius" value="${chassis_props['wheel_radius']['front']}" />
-    <xacro:property name="rear_wheel_radius" value="${chassis_props['wheel_radius']['rear']}" />
-    <xacro:property name="front_wheel_width" value="${chassis_props['wheel_width']['front']}" />
-    <xacro:property name="rear_wheel_width" value="${chassis_props['wheel_width']['rear']}" />
+    <xacro:property name="front_wheel_radius" value="${props['geometry']['front_axle']['wheels']['radius']}" />
+    <xacro:property name="rear_wheel_radius" value="${props['geometry']['rear_axle']['wheels']['radius']}" />
+    <xacro:property name="front_wheel_width" value="${props['geometry']['front_axle']['wheels']['width']}" />
+    <xacro:property name="rear_wheel_width" value="${props['geometry']['rear_axle']['wheels']['width']}" />
     <xacro:property name="front_wheel_mass" value="20." />
     <xacro:property name="rear_wheel_mass" value="20." />
@@ -50,7 +44,7 @@
     <xacro:property name="wheel_width" value="${front_wheel_width}" />
     <!-- Wheel Mounting Positions -->
-    <xacro:property name="ground_clearance" value="${chassis_props['ground_clearance']}"/>
-    <xacro:property name="front_wheel_y_offset" value="${chassis_props['hub_carrier_offset']['front']}" />
-    <xacro:property name="rear_wheel_y_offset" value="${chassis_props['hub_carrier_offset']['rear']}" />
+    <xacro:property name="ground_clearance" value="${props['geometry']['ground_clearance']}"/>
+    <xacro:property name="front_wheel_y_offset" value="${props['geometry']['rear_axle']['wheels']['hub_carrier_offset']}" />
+    <xacro:property name="rear_wheel_y_offset" value="${props['geometry']['rear_axle']['wheels']['hub_carrier_offset']}" />
     <xacro:property name="chassis_height" value="${min(front_wheel_radius,rear_wheel_radius)}" />
   <xacro:macro name="effibote3" params="use_sim prefix">

File: effibote3_description/urdf/old/effibote3.urdf.xacro (robot description, xacro)
@@ -4,12 +4,11 @@
   <xacro:arg name="use_sim" default="true" />
   <xacro:arg name="controller_conf_yaml_file" default=""/>
-  <xacro:property name="prefix" value="$(arg prefix)"/>
-  <xacro:property name="controller_conf_yaml_file" value="$(arg controller_conf_yaml_file)"/>
+<!--  <xacro:property name="prefix" value="$(arg prefix)"/>-->
+<!--  <xacro:property name="controller_conf_yaml_file" value="$(arg controller_conf_yaml_file)"/>-->
   <xacro:include filename="$(find effibote3_description)/urdf/effibote3.xacro" />
   <xacro:effibote3 use_sim="$(arg use_sim)" prefix="$(arg prefix)"/>
   <gazebo>
     <plugin filename="libgazebo_ros2_control.so" name="gazebo_ros2_control">
-       <parameters>${controller_conf_yaml_file}</parameters>
-<!--       <parameters>${arg controller_conf_yaml_file}</parameters>-->
+       <parameters>${arg controller_conf_yaml_file}</parameters>
     </plugin>
   </gazebo>

Commit message: gazebo launch works

File: effibote3_description/urdf/effibote3.xacro (robot description, xacro)
@@ -45,5 +45,5 @@
     <!-- Wheel Mounting Positions -->
     <xacro:property name="ground_clearance" value="${props['geometry']['ground_clearance']}"/>
-    <xacro:property name="front_wheel_y_offset" value="${props['geometry']['rear_axle']['wheels']['hub_carrier_offset']}" />
+    <xacro:property name="front_wheel_y_offset" value="${props['geometry']['front_axle']['wheels']['hub_carrier_offset']}" />
     <xacro:property name="rear_wheel_y_offset" value="${props['geometry']['rear_axle']['wheels']['hub_carrier_offset']}" />
     <xacro:property name="chassis_height" value="${min(front_wheel_radius,rear_wheel_radius)}" />

Commit message: effibot description : change hardware plugin name in live mode

File: effibote3_description/urdf/effibote3.xacro (robot description, xacro)
@@ -50,5 +50,5 @@
    <!-- Ros2 control hardware plugin -->
    <xacro:property name="simulation_hardware_plugin" value="romea_mobile_base_gazebo/GazeboSystemInterface4WD"/>
-   <xacro:property name="live_hardware_plugin" value="effibote3_hardware/Effibote3Hardware"/>
+   <xacro:property name="live_hardware_plugin" value="effibote3_hardware/EffibotE3Hardware"/>
   <xacro:macro name="effibote3" params="mode prefix">
     <xacro:chassis>

Commit message: description : update xacro files

File: effibote3_description/urdf/effibote3.xacro (robot description, xacro)
@@ -2,6 +2,6 @@
 <robot name="effibote3" xmlns:xacro="http://ros.org/wiki/xacro">
     <xacro:property name="M_PI" value="3.14159"/>
-    <xacro:include filename="$(find romea_mobile_base_description)/urdf/4WD_chassis.xacro" />
-    <xacro:include filename="$(find romea_mobile_base_description)/ros2_control/4WD.ros2_control.xacro"/>
+    <xacro:include filename="$(find romea_mobile_base_description)/urdf/base4WD.chassis.xacro" />
+    <xacro:include filename="$(find romea_mobile_base_description)/ros2_control/base4WD.ros2_control.xacro"/>
     <xacro:property name="conf" value="$(find effibote3_description)/config/effibote3.yaml" />
     <xacro:property name="props" value="${load_yaml(conf)['/**']['ros__parameters']['base_info']}" />
@@ -22,7 +22,11 @@
     <xacro:property name="rear_right_wheel_spinning_joint" value="${props['joints']['rear_right_wheel_spinning_joint_name']}" />
     <!-- Base Properties -->
+    <xacro:property name="ground_clearance" value="${props['geometry']['ground_clearance']}"/>
     <xacro:property name="aabb_length" value="${props['geometry']['aabb']['length']}" />
     <xacro:property name="aabb_width" value="${props['geometry']['aabb']['width']}" />
     <xacro:property name="aabb_height" value="${props['geometry']['aabb']['height']}" />
+    <xacro:property name="aabb_center_x" value="${props['geometry']['aabb']['center'][0]}" />
+    <xacro:property name="aabb_center_y" value="${props['geometry']['aabb']['center'][1]}" />
+    <xacro:property name="aabb_center_z" value="${props['geometry']['aabb']['center'][2]}" />
     <xacro:property name="wheelbase" value="${props['geometry']['axles_distance']}"/>
     <xacro:property name="front_track" value="${props['geometry']['front_axle']['wheels_distance']}"/>
@@ -44,5 +48,4 @@
     <xacro:property name="wheel_width" value="${front_wheel_width}" />
     <!-- Wheel Mounting Positions -->
-    <xacro:property name="ground_clearance" value="${props['geometry']['ground_clearance']}"/>
     <xacro:property name="front_wheel_y_offset" value="${props['geometry']['front_axle']['wheels']['hub_carrier_offset']}" />
     <xacro:property name="rear_wheel_y_offset" value="${props['geometry']['rear_axle']['wheels']['hub_carrier_offset']}" />
@@ -57,4 +60,5 @@
             <box size="${aabb_length} ${aabb_width} ${aabb_height}"/>
           </geometry>
+          <origin xyz="${aabb_center_x-body_reference_x} ${aabb_center_y}  ${aabb_center_z-chassis_height}" rpy="0 0 0" />
           <material name="grey">
             <color rgba="0.6 0.6 0.6 1"/>
