Commit message: effibote3 description : add controller_conf_file and use_sim arguments into xacro files

File: effibote3_description/urdf/effibote3.urdf.xacro (robot description, xacro)
@@ -1,9 +1,14 @@
 <?xml version='1.0' encoding='utf-8'?>
 <robot name="effibote3" xmlns:xacro="http://www.ros.org/wiki/xacro">
-  <xacro:property name="prefix" value="" />
+  <xacro:arg name="prefix" default="" />
+  <xacro:arg name="use_sim" default="true" />
+  <xacro:arg name="controller_conf_yaml_file" default=""/>
+  <xacro:property name="prefix" value="$(arg prefix)"/>
+  <xacro:property name="controller_conf_yaml_file" value="$(arg controller_conf_yaml_file)"/>
   <xacro:include filename="$(find effibote3_description)/urdf/effibote3.xacro" />
-  <xacro:effibote3/>
+  <xacro:effibote3 use_sim="$(arg use_sim)" prefix="$(arg prefix)"/>
   <gazebo>
-    <plugin filename="libgazebo_ros_control2.so" name="gazebo_ros2_control">
+    <plugin filename="libgazebo_ros2_control.so" name="gazebo_ros2_control">
+    <parameters>${controller_conf_yaml_file}</parameters>
     </plugin>
   </gazebo>

File: effibote3_description/urdf/effibote3.xacro (robot description, xacro)
@@ -54,5 +54,5 @@
     <xacro:property name="rear_wheel_y_offset" value="${chassis_props['hub_carrier_offset']['rear']}" />
     <xacro:property name="chassis_height" value="${min(front_wheel_radius,rear_wheel_radius)}" />
-  <xacro:macro name="effibote3">
+  <xacro:macro name="effibote3" params="use_sim prefix">
     <xacro:chassis>
         <visual>
@@ -67,5 +67,5 @@
         <cylinder length="${wheel_width}" radius="${wheel_radius}"/>
     </xacro:chassis>
-    <xacro:base_control/>
+    <xacro:base_control use_sim="${use_sim}"/>
   </xacro:macro>
 </robot>

Commit message: effibote3_description : reafactoring due to changes into mobile_base_description package

File: effibote3_description/urdf/effibote3.urdf.xacro (robot description, xacro)
@@ -2,10 +2,10 @@
 <robot name="effibote3" xmlns:xacro="http://www.ros.org/wiki/xacro">
   <xacro:arg name="prefix" default="" />
-  <xacro:arg name="use_sim" default="true" />
+  <xacro:arg name="mode" default="simulation" />
   <xacro:arg name="controller_conf_yaml_file" default=""/>
   <xacro:property name="prefix" value="$(arg prefix)"/>
   <xacro:property name="controller_conf_yaml_file" value="$(arg controller_conf_yaml_file)"/>
   <xacro:include filename="$(find effibote3_description)/urdf/effibote3.xacro" />
-  <xacro:effibote3 use_sim="$(arg use_sim)" prefix="$(arg prefix)"/>
+  <xacro:effibote3 mode="$(arg mode)" prefix="$(arg prefix)"/>
   <gazebo>
     <plugin filename="libgazebo_ros2_control.so" name="gazebo_ros2_control">

File: effibote3_description/urdf/effibote3.xacro (robot description, xacro)
@@ -48,5 +48,8 @@
     <xacro:property name="rear_wheel_y_offset" value="${props['geometry']['rear_axle']['wheels']['hub_carrier_offset']}" />
     <xacro:property name="chassis_height" value="${min(front_wheel_radius,rear_wheel_radius)}" />
-  <xacro:macro name="effibote3" params="use_sim prefix">
+   <!-- Ros2 control hardware plugin -->
+   <xacro:property name="simulation_hardware_plugin" value="romea_mobile_base_gazebo/GazeboSystemInterface4WD"/>
+   <xacro:property name="live_hardware_plugin" value="effibote3_hardware/Effibote3Hardware"/>
+  <xacro:macro name="effibote3" params="mode prefix">
     <xacro:chassis>
         <visual>
@@ -61,5 +64,7 @@
         <cylinder length="${wheel_width}" radius="${wheel_radius}"/>
     </xacro:chassis>
-    <xacro:base_control use_sim="${use_sim}"/>
+    <xacro:if value="${mode == 'simulation' or mode == 'live'}">
+       <xacro:base_control mode="${mode}"/>
+    </xacro:if>
   </xacro:macro>
 </robot>

Commit message: first version of hardware plugin
Signed-off-by: jean.laneurit <jean.laneurit@inrae.fr>

File: effibote3_description/urdf/effibote3.urdf.xacro (robot description, xacro)
@@ -1,15 +1,19 @@
 <?xml version='1.0' encoding='utf-8'?>
 <robot name="effibote3" xmlns:xacro="http://www.ros.org/wiki/xacro">
-  <xacro:arg name="prefix" default="" />
+  <xacro:arg name="prefix" default="effibote3_" />
   <xacro:arg name="mode" default="simulation" />
-  <xacro:arg name="controller_conf_yaml_file" default=""/>
-  <xacro:property name="prefix" value="$(arg prefix)"/>
-  <xacro:property name="controller_conf_yaml_file" value="$(arg controller_conf_yaml_file)"/>
+  <xacro:arg name="base_name" default="base" />
+  <xacro:arg name="ros2_control_config_urdf_file" default="" />
+  <xacro:arg name="controller_manager_config_yaml_file" default="" />
+  <xacro:arg name="ros_prefix" default="/effibote3/" />
   <xacro:include filename="$(find effibote3_description)/urdf/effibote3.xacro" />
-  <xacro:effibote3 mode="$(arg mode)" prefix="$(arg prefix)"/>
+  <xacro:effibote3 mode="$(arg mode)" prefix="$(arg prefix)" />
   <gazebo>
-    <plugin filename="libgazebo_ros2_control.so" name="gazebo_ros2_control">
-       <parameters>${controller_conf_yaml_file}</parameters>
-<!--       <parameters>${arg controller_conf_yaml_file}</parameters>-->
+    <plugin filename="libromea_gazebo_ros2_control.so" name="gazebo_ros2_control">
+      <ros2_control_config_file>$(arg ros2_control_config_urdf_file)</ros2_control_config_file>
+      <controller_manager_config_file>$(arg controller_manager_config_yaml_file)</controller_manager_config_file>
+      <ros>
+        <namespace>$(arg ros_prefix)$(arg base_name)</namespace>
+      </ros>
     </plugin>
   </gazebo>

File: effibote3_description/urdf/effibote3.xacro (robot description, xacro)
@@ -1,74 +1,109 @@
 <?xml version="1.0"?>
 <robot name="effibote3" xmlns:xacro="http://ros.org/wiki/xacro">
-    <xacro:property name="M_PI" value="3.14159"/>
-    <xacro:include filename="$(find romea_mobile_base_description)/urdf/base4WD.chassis.xacro" />
-    <xacro:include filename="$(find romea_mobile_base_description)/ros2_control/base4WD.ros2_control.xacro"/>
-    <xacro:property name="conf" value="$(find effibote3_description)/config/effibote3.yaml" />
-    <xacro:property name="props" value="${load_yaml(conf)['/**']['ros__parameters']['base_info']}" />
-    <!-- Link names -->
-    <xacro:property name="base_link" value="${props['links']['base_link_name']}" />
-    <xacro:property name="base_footprint_link" value="${props['links']['base_footprint_link_name']}" />
-    <xacro:property name="inertial_link" value="${props['links']['inertial_link_name']}" />
-    <xacro:property name="front_left_wheel_spinning_link" value="${props['links']['front_left_wheel_spinning_link_name']}" />
-    <xacro:property name="front_right_wheel_spinning_link" value="${props['links']['front_right_wheel_spinning_link_name']}" />
-    <xacro:property name="rear_left_wheel_spinning_link" value="${props['links']['rear_left_wheel_spinning_link_name']}" />
-    <xacro:property name="rear_right_wheel_spinning_link" value="${props['links']['rear_right_wheel_spinning_link_name']}" />
-    <!-- Joint names -->
-    <xacro:property name="base_footprint_joint" value="${props['joints']['base_footprint_joint_name']}" />
-    <xacro:property name="inertial_joint" value="${props['joints']['inertial_joint_name']}" />
-    <xacro:property name="front_left_wheel_spinning_joint" value="${props['joints']['front_left_wheel_spinning_joint_name']}" />
-    <xacro:property name="front_right_wheel_spinning_joint" value="${props['joints']['front_right_wheel_spinning_joint_name']}" />
-    <xacro:property name="rear_left_wheel_spinning_joint" value="${props['joints']['rear_left_wheel_spinning_joint_name']}" />
-    <xacro:property name="rear_right_wheel_spinning_joint" value="${props['joints']['rear_right_wheel_spinning_joint_name']}" />
-    <!-- Base Properties -->
-    <xacro:property name="ground_clearance" value="${props['geometry']['ground_clearance']}"/>
-    <xacro:property name="aabb_length" value="${props['geometry']['aabb']['length']}" />
-    <xacro:property name="aabb_width" value="${props['geometry']['aabb']['width']}" />
-    <xacro:property name="aabb_height" value="${props['geometry']['aabb']['height']}" />
-    <xacro:property name="aabb_center_x" value="${props['geometry']['aabb']['center'][0]}" />
-    <xacro:property name="aabb_center_y" value="${props['geometry']['aabb']['center'][1]}" />
-    <xacro:property name="aabb_center_z" value="${props['geometry']['aabb']['center'][2]}" />
-    <xacro:property name="wheelbase" value="${props['geometry']['axles_distance']}"/>
-    <xacro:property name="front_track" value="${props['geometry']['front_axle']['wheels_distance']}"/>
-    <xacro:property name="rear_track" value="${props['geometry']['rear_axle']['wheels_distance']}"/>
-    <xacro:property name="mass_base" value="${props['inertia']['mass']}" />
-    <xacro:property name="mass_center_x" value="${props['inertia']['center'][0]}" />
-    <xacro:property name="mass_center_y" value="${props['inertia']['center'][1]}" />
-    <xacro:property name="mass_center_z" value="${props['inertia']['center'][2]}" />
-    <xacro:property name="maximal_wheel_speed" value="${props['wheels_speed_control']['command']['maximal_speed']}"/>
-    <xacro:property name="body_reference_x" value="${props['control_point'][0]}" />
-    <!-- Wheel Properties -->
-    <xacro:property name="front_wheel_radius" value="${props['geometry']['front_axle']['wheels']['radius']}" />
-    <xacro:property name="rear_wheel_radius" value="${props['geometry']['rear_axle']['wheels']['radius']}" />
-    <xacro:property name="front_wheel_width" value="${props['geometry']['front_axle']['wheels']['width']}" />
-    <xacro:property name="rear_wheel_width" value="${props['geometry']['rear_axle']['wheels']['width']}" />
-    <xacro:property name="front_wheel_mass" value="20." />
-    <xacro:property name="rear_wheel_mass" value="20." />
-    <xacro:property name="wheel_radius" value="${front_wheel_radius}" />
-    <xacro:property name="wheel_width" value="${front_wheel_width}" />
-    <!-- Wheel Mounting Positions -->
-    <xacro:property name="front_wheel_y_offset" value="${props['geometry']['front_axle']['wheels']['hub_carrier_offset']}" />
-    <xacro:property name="rear_wheel_y_offset" value="${props['geometry']['rear_axle']['wheels']['hub_carrier_offset']}" />
-    <xacro:property name="chassis_height" value="${min(front_wheel_radius,rear_wheel_radius)}" />
-   <!-- Ros2 control hardware plugin -->
-   <xacro:property name="simulation_hardware_plugin" value="romea_mobile_base_gazebo/GazeboSystemInterface4WD"/>
-   <xacro:property name="live_hardware_plugin" value="effibote3_hardware/EffibotE3Hardware"/>
+  <!-- <xacro:property name="M_PI" value="3.14159" /> -->
+  <xacro:include filename="$(find romea_mobile_base_description)/urdf/base4WD.chassis.xacro" />
+  <xacro:include filename="$(find effibote3_description)/urdf/visual/chassis.xacro" />
+  <xacro:include filename="$(find effibote3_description)/urdf/visual/wheels.xacro" />
+  <xacro:property name="conf" value="$(find effibote3_description)/config/effibote3.yaml" />
+  <xacro:property name="props" value="${load_yaml(conf)}" />
+  <!-- Link names -->
+  <xacro:property name="base_link"
+    value="${props['links']['base_link_name']}" />
+  <xacro:property name="base_footprint_link"
+    value="${props['links']['base_footprint_link_name']}" />
+  <xacro:property name="inertial_link"
+    value="${props['links']['inertial_link_name']}" />
+  <xacro:property name="front_left_wheel_spinning_link"
+    value="${props['links']['front_left_wheel_spinning_link_name']}" />
+  <xacro:property name="front_right_wheel_spinning_link"
+    value="${props['links']['front_right_wheel_spinning_link_name']}" />
+  <xacro:property name="rear_left_wheel_spinning_link"
+    value="${props['links']['rear_left_wheel_spinning_link_name']}" />
+  <xacro:property name="rear_right_wheel_spinning_link"
+    value="${props['links']['rear_right_wheel_spinning_link_name']}" />
+  <!-- Joint names -->
+  <xacro:property name="base_footprint_joint"
+    value="${props['joints']['base_footprint_joint_name']}" />
+  <xacro:property name="inertial_joint"
+    value="${props['joints']['inertial_joint_name']}" />
+  <xacro:property name="front_left_wheel_spinning_joint"
+    value="${props['joints']['front_left_wheel_spinning_joint_name']}" />
+  <xacro:property name="front_right_wheel_spinning_joint"
+    value="${props['joints']['front_right_wheel_spinning_joint_name']}" />
+  <xacro:property name="rear_left_wheel_spinning_joint"
+    value="${props['joints']['rear_left_wheel_spinning_joint_name']}" />
+  <xacro:property name="rear_right_wheel_spinning_joint"
+    value="${props['joints']['rear_right_wheel_spinning_joint_name']}" />
+  <!-- Base Properties -->
+  <xacro:property name="aabb_length"
+    value="${props['geometry']['aabb']['length']}" />
+  <xacro:property name="aabb_width"
+    value="${props['geometry']['aabb']['width']}" />
+  <xacro:property name="aabb_height"
+    value="${props['geometry']['aabb']['height']}" />
+  <xacro:property name="aabb_center_x"
+    value="${props['geometry']['aabb']['center'][0]}" />
+  <xacro:property name="aabb_center_y"
+    value="${props['geometry']['aabb']['center'][1]}" />
+  <xacro:property name="aabb_center_z"
+    value="${props['geometry']['aabb']['center'][2]}" />
+  <xacro:property name="wheelbase"
+    value="${props['geometry']['axles_distance']}" />
+  <xacro:property name="front_track"
+    value="${props['geometry']['front_axle']['wheels_distance']}" />
+  <xacro:property name="rear_track"
+    value="${props['geometry']['rear_axle']['wheels_distance']}" />
+  <xacro:property name="mass_base"
+    value="${props['inertia']['mass']}" />
+  <xacro:property name="mass_center_x"
+    value="${props['inertia']['center'][0]}" />
+  <xacro:property name="mass_center_y"
+    value="${props['inertia']['center'][1]}" />
+  <xacro:property name="mass_center_z"
+    value="${props['inertia']['center'][2]}" />
+  <xacro:property name="ground_clearance"
+    value="${props['geometry']['ground_clearance']}" />
+  <xacro:property name="body_reference_x"
+    value="${props['control_point'][0]}" />
+  <xacro:property name="maximal_wheel_speed"
+    value="${props['wheels_speed_control']['command']['maximal_speed']}" />
+  <xacro:property name="body_reference_x" value="${props['control_point'][0]}" />
+  <!-- Wheel Properties -->
+  <xacro:property name="front_wheel_y_offset"
+    value="${props['geometry']['front_axle']['wheels']['hub_carrier_offset']}" />
+  <xacro:property name="rear_wheel_y_offset"
+    value="${props['geometry']['rear_axle']['wheels']['hub_carrier_offset']}" />
+  <xacro:property name="wheel_y_offset"
+    value="${front_wheel_y_offset}" />
+  <xacro:property name="front_hub_carrier_offset"
+    value="${props['geometry']['front_axle']['wheels']['hub_carrier_offset']}" />
+  <xacro:property name="rear_hub_carrier_offset"
+    value="${props['geometry']['rear_axle']['wheels']['hub_carrier_offset']}" />
+  <xacro:property name="front_wheel_radius"
+    value="${props['geometry']['front_axle']['wheels']['radius']}" />
+  <xacro:property name="rear_wheel_radius"
+    value="${props['geometry']['rear_axle']['wheels']['radius']}" />
+  <xacro:property name="front_wheel_width"
+    value="${props['geometry']['front_axle']['wheels']['width']}" />
+  <xacro:property name="rear_wheel_width"
+    value="${props['geometry']['rear_axle']['wheels']['width']}" />
+  <xacro:property name="maximal_wheel_speed"
+    value="${props['wheels_speed_control']['command']['maximal_speed']}" />
+  <xacro:property name="wheel_mass" value="5." />
+  <xacro:property name="front_wheel_mass" value="5." />
+  <xacro:property name="rear_wheel_mass" value="5." />
+  <xacro:property name="chassis_height"
+    value="${min(front_wheel_radius,rear_wheel_radius)}" />
+  <!-- <xacro:property name="wheel_radius" value="${front_wheel_radius}" /> -->
+  <!-- <xacro:property name="wheel_width" value="${front_wheel_width}" /> -->
+  <!-- Wheel Mounting Positions -->
   <xacro:macro name="effibote3" params="mode prefix">
     <xacro:chassis>
-        <visual>
-          <geometry>
-            <box size="${aabb_length} ${aabb_width} ${aabb_height}"/>
-          </geometry>
-          <origin xyz="${aabb_center_x-body_reference_x} ${aabb_center_y}  ${aabb_center_z-chassis_height}" rpy="0 0 0" />
-          <material name="grey">
-            <color rgba="0.6 0.6 0.6 1"/>
-          </material>
-        </visual>
-        <!-- visual wheel -->
-        <cylinder length="${wheel_width}" radius="${wheel_radius}"/>
+      <xacro:chassis_visual />
+      <xacro:front_left_wheel_visual />
+      <xacro:front_right_wheel_visual />
+      <xacro:rear_left_wheel_visual />
+      <xacro:rear_right_wheel_visual />
     </xacro:chassis>
-    <xacro:if value="${mode == 'simulation' or mode == 'live'}">
-       <xacro:base_control mode="${mode}"/>
-    </xacro:if>
   </xacro:macro>
 </robot>
